Commit message: added rtv moveit commanding

File: moveit2_ws/src/unitree_moveit_config/config/g1_29dof_rev_1_0_with_inspire_hand_FTP.ros2_control.xacro (robot description, xacro)
@@ -9,4 +9,25 @@
                 <param name="joint_states_topic">/lowstate_joint_states</param>
             </hardware>
+            <joint name="waist_yaw_joint">
+                <command_interface name="position"/>
+                <state_interface name="position">
+                    <!-- <param name="initial_value">${initial_positions['right_shoulder_pitch_joint']}</param> -->
+                </state_interface>
+                <state_interface name="velocity"/>
+            </joint>
+            <joint name="waist_roll_joint">
+                <command_interface name="position"/>
+                <state_interface name="position">
+                    <!-- <param name="initial_value">${initial_positions['right_shoulder_pitch_joint']}</param> -->
+                </state_interface>
+                <state_interface name="velocity"/>
+            </joint>
+            <joint name="waist_pitch_joint">
+                <command_interface name="position"/>
+                <state_interface name="position">
+                    <!-- <param name="initial_value">${initial_positions['right_shoulder_pitch_joint']}</param> -->
+                </state_interface>
+                <state_interface name="velocity"/>
+            </joint>
             <joint name="left_shoulder_pitch_joint">
                 <command_interface name="position"/>
